File: hardware/v2.0/Patch-Prop.sch (EAGLE design)
At the start: 50 parts, among them IC1 TPS77033, IC2 ATMEGA168, IC3 XBEE, IC4 MMA8452Q, U1 MCP73831, U2 MCP1253, X1 USBSMD

Commit message: Added LED driver in MSOP8 package + raw brd file
Parts:
- added U$1: W2RV005RM, Sparky:W2RV005RM
Connections:
- removed net N$3: LED3.BLUE_A, LED3.GREEN_A, LED3.RED_A, LED4.BLUE_A, LED4.GREEN_A, LED4.RED_A, LED5.BLUE_A, LED5.GREEN_A, LED5.RED_A, LED6.BLUE_A, LED6.GREEN_A, LED6.RED_A
- new net BLUE_OUT: LED3.BLUE_C, LED4.BLUE_C, LED5.BLUE_C, LED6.BLUE_C, U$1.OUT1
- new net GREEN_OUT: LED3.GREEN_C, LED4.GREEN_C, LED5.GREEN_C, LED6.GREEN_C, U$1.OUT2
- new net RED_OUT: LED3.RED_C, LED4.RED_C, LED5.RED_C, LED6.RED_C, U$1.OUT3
- net BLUE: now also U$1.IN1
- net GND: now also U$1.GND
- net GREEN: now also U$1.IN2
- net RED: now also U$1.IN3
- net V+: now also LED3.BLUE_A, LED3.GREEN_A, LED3.RED_A, LED4.BLUE_A, LED4.GREEN_A, LED4.RED_A, LED5.BLUE_A, LED5.GREEN_A, LED5.RED_A, LED6.BLUE_A, LED6.GREEN_A, LED6.RED_A, U$1.VCC
Other:
- note added: "Questions: -Should the vibe have a connector? -Should the prox have a connector? It could just have header holes and we solder a cable with a connector -Do we want to use the shtdwn for the stepup or power good -Double check we are on PWM channels -Double check stepup select and shtdwn -Double check connector direction for battery and prox sensor -Do we want a PMC? -Check pin layout power consump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"
- note removed: "Questions: -Should the vibe have a connector? -Should the prox have a connector? It could just have header holes and we solder a cable with a connector -Do we want to use the shtdwn for the stepup or power good -Double check we are on PWM channels -Double check stepup select and shtdwn -Double check connector direction for battery and prox sensor"

Commit message: Tweaking naming and notes
Parts:
- removed R9: 470, SparkFun:RESISTOR0402-RES
- removed U1: MCP73831, SparkFun:MCP73831SMD
- added IC5: MCP1253, CH_Microchip:MCP1253
- added R7: 10k, rcl:R-US_R0603
- C1, C5: device rcl:C-USC0603 -> CH_passive:CAP0603
- C10, C9: value 4.7uF -> 0.1uF; device SparkFun:CAP0402-CAP -> rcl:C-USC0603
- C11: value 0.1uF -> 4.7uF
- C12: value 1uF -> .1uF; device CH_passive:CAP0603 -> rcl:C-USC0603
- C13: device CH_passive:CAP0603 -> rcl:C-USC0603
- C14: value 10uF -> .1uF; device CH_passive:CAP0603 -> rcl:C-USC0603
- C3: value .1uF -> 1uF
- C4: value .1uF -> 10uF; device rcl:C-USC0603 -> CH_passive:CAP0603
- C7: value 0.1uF -> 4.7uF; device rcl:C-USC0603 -> SparkFun:CAP0402-CAP
- C8: device rcl:C-USC0603 -> SparkFun:CAP0402-CAP
- IC2: value ATMEGA168 -> XBEE; device SparkFun:ATMEGA168 -> adafruit:XBEE
- IC3: value XBEE -> MMA8452Q; device adafruit:XBEE -> eski-ic:MMA8452Q
- IC4: value MMA8452Q -> ATMEGA168; device eski-ic:MMA8452Q -> SparkFun:ATMEGA168
- JP2: device SparkFun-Connectors:M03 -> SparkFun-Connectors:M02-JST-2MM-SMT
- JP3: device SparkFun-Connectors:M02-JST-2MM-SMT -> SparkFun-Connectors:M02PTH
- JP5: device SparkFun-Connectors:M02-JST-2MM-SMT -> SparkFun-Connectors:M03
- JP7: device SparkFun-Connectors:M02PTH -> SparkFun-Connectors:M02-JST-2MM-SMT
- R2: value 10k -> 470; device rcl:R-US_R0603 -> SparkFun:RESISTOR0402-RES
- R3: value 470 -> 10k
- R4: value 10k -> 2K; device rcl:R-US_R0603 -> SparkFun:RESISTOR0402-RES
- R5: value 2K -> 470; device SparkFun:RESISTOR0402-RES -> rcl:R-US_R0603
- U2: value MCP1253 -> MCP73831; device CH_Microchip:MCP1253 -> SparkFun:MCP73831SMD
- renumbered D4 to D1, LED7 to LED1, R12 to R6, U$1 to IC6
Connections:
- net +3V3: now also C13.1, C14.1, C4.2, C9.1, IC2.VCC, IC3.VDD, IC3.VDDIO, IC4.AVCC, IC4.VCC@1, IC4.VCC@2, IC5./SHDN, IC5.VIN, R5.2, R7.2; no longer C13.2, C5.1, C6.1, C8.1, IC2.AVCC, IC2.VCC@1, IC2.VCC@2, IC3.VCC, IC4.VDD, IC4.VDDIO, R3.2, R4.2, U2./SHDN, U2.VIN
- net +5V: now also JP5.3; no longer JP2.3
- net BLUE: now also IC4.PB2(SS/OC1B); no longer IC2.PB2(SS/OC1B)
- net DTR: now also C12.1; no longer C4.1
- net GND: now also C13.2, C14.2, C3.2, C4.1, C5.1, IC2.GND, IC3.GND1, IC3.GND2, IC3.GND3, IC3.SA0, IC4.AGND, IC4.GND@1, IC4.GND@2, IC5.GND, IC5.SELECT, JP3.1, JP5.2, R3.1, R4.2, U2.VSS; no longer C1.2, C13.1, C14.1, C5.2, C6.2, IC2.AGND, IC2.GND@1, IC2.GND@2, IC3.GND, IC4.GND1, IC4.GND2, IC4.GND3, IC4.SA0, JP3.2, JP6.1, R2.1, R5.2, U1.VSS, U2.GND, U2.SELECT
- net GREEN: now also IC4.PD5(T1); no longer IC2.PD5(T1)
- net INT0: now also IC4.PD2(INT0); no longer IC2.PD2(INT0)
- net INT1: now also IC3.INT1, IC4.PD3(INT1); no longer IC2.PD3(INT1), IC4.INT1
- net INT2: now also IC3.INT2; no longer IC4.INT2
- net MISO: now also IC4.PB4(MISO); no longer IC2.PB4(MISO)
- net MOSI: now also IC4.PB3(MOSI/OC2); no longer IC2.PB3(MOSI/OC2)
- net N$1: now also C6.1, IC2.AD3/DIO3, SJ2.2; no longer C3.1, IC3.AD3/DIO3, SJ1.2
- net N$10: now also C5.2, IC5.VOUT; no longer C14.2, U2.VOUT
- net N$11: now also R4.1, U2.PROG; no longer R5.1, U1.PROG
- net N$14: now also R2.1, U2.STAT; no longer R9.1, U1.STAT
- net N$16: now also C10.1, IC3.BYP; no longer C7.1, IC4.BYP
- net N$18: now also IC2.CTS/DIO7, SJ2.1; no longer IC3.CTS/DIO7, SJ1.1
- net N$19: now also IC2.RESET, SJ1.1; no longer IC3.RESET, SJ2.1
- net N$2: now also C6.2, R3.2; no longer C3.2, R2.2
- net N$5: now also R5.1; no longer R3.1
- net N$6: now also C1.1, IC5.C-; no longer C12.1, U2.C-
- net N$7: now also C1.2, IC5.C+; no longer C12.2, U2.C+
- net N$8: now also R2.2; no longer R9.2
- net PGOOD: now also IC5.PGOOD; no longer U2.PGOOD
- net PROXIN: now also IC4.PC0(ADC0), JP5.1; no longer IC2.PC0(ADC0), JP2.1
- net RED: now also IC4.PB1(OC1A); no longer IC2.PB1(OC1A)
- net RESET: now also C12.2, IC4.PC6(/RESET), R7.1, SJ1.2; no longer C4.2, IC2.PC6(/RESET), R4.1, SJ2.2
- net RXD: now also IC2.DOUT, IC4.PD0(RXD); no longer IC2.PD0(RXD), IC3.DOUT
- net SCK: now also IC4.PB5(SCK); no longer IC2.PB5(SCK)
- net SCL: now also IC3.SCL, IC4.PC5(ADC5/SCL); no longer IC2.PC5(ADC5/SCL), IC4.SCL
- net SDA: now also IC3.SDA, IC4.PC4(ADC4/SDA); no longer IC2.PC4(ADC4/SDA), IC4.SDA
- net STATUS: now also IC4.PD7(AIN1); no longer IC2.PD7(AIN1)
- net TXD: now also IC2.DIN, IC4.PD1(TXD); no longer IC2.PD1(TXD), IC3.DIN
- net USB_VIN: now also C7.1, JP3.2, U2.VIN; no longer C9.1, JP6.2, U1.VIN
- net V+: now also C3.1, C8.1, JP2.1, JP6.1, U2.VBAT; no longer C1.1, C10.1, JP3.1, JP5.1, U1.VBAT
- net VIBE: now also JP6.2; no longer JP5.2
- net VIBE_CONTROL: now also IC4.PB0(ICP); no longer IC2.PB0(ICP)
Other:
- moved on the sheet: C1, C10, C11, C12, C13, C14, C3, C4, C5, C6, C7, C8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

Commit message: Working on PCB
Parts:
- removed C7, C8: 4.7uF, SparkFun:CAP0402-CAP
- removed JP3: (no value), SparkFun-Connectors:M02PTH
- added C15, C16: 4.7uF, rcl:C-USC0603
- C1, C4, C5: device CH_passive:CAP0603 -> rcl:C-USC0603
- D1: value Yellow -> (none); device SparkFun:LED0603 -> led:LEDCHIPLED_0805
- R1: device CH_passive:RESISTOR0603 -> rcl:R-US_R0603
- R2: device SparkFun:RESISTOR0402-RES -> rcl:R-US_R0603
- R4: value 2K -> 2k; device SparkFun:RESISTOR0402-RES -> rcl:R-US_R0603
Connections:
- net +3V3: now also C4.1; no longer C4.2
- net GND: now also C15.2, C16.2, C4.2, C5.2; no longer C4.1, C5.1, C7.2, C8.2, JP3.1
- net N$10: now also C5.1, R1.1; no longer C5.2, R1.2
- net PGOOD: now also R1.2; no longer R1.1
- net USB_VIN: now also C16.1; no longer C7.1, JP3.2
- net V+: now also C15.1; no longer C8.1
Other:
- moved on the sheet: C4, C5, R1

Commit message: Tentative part layout for propinquity board
Parts:
- removed ICSP: (no value), pinhead:PINHD-2X3
- removed JP1: (no value), SparkFun-Connectors:M02PTH
- removed JP4: (no value), SparkFun:ARDUINO_SERIAL_PROGRAMSMD
- removed JP7: (no value), SparkFun-Connectors:M02-JST-2MM-SMT
- removed RESET: (no value), SparkFun:TAC_SWITCHPTH
- added C7: 4.7uF, rcl:C-USC0603
- added ISP1: (no value), balto:ISP-AVR910SMD
- added JP3: (no value), SparkFun-Connectors:M03PTH
- added SJ3: SOLDERJUMPERNO, SparkFun:SOLDERJUMPERNO
- JP5: device SparkFun-Connectors:M03 -> SparkFun-Connectors:ARDUINO_SERIAL_PROGRAMPTH
- SHARP: value GP2D12TH -> GP2D12_OUTLINE; device Sparky:GP2D12TH -> Sparky:GP2D12_OUTLINE
Connections:
- removed net INT2: IC3.INT2
- net +3V3: now also JP5.VCC; no longer ICSP.2, JP4.VCC
- net +5V: now also JP3.3; no longer JP5.3, SHARP.VCC
- net DTR: now also JP5.DTR; no longer JP4.DTR
- net GND: now also C7.2, JP3.2, JP5.CTS, JP5.GND, SJ3.1; no longer ICSP.6, JP1.2, JP4.CTS, JP4.GND, JP5.2, RESET.3, RESET.4, SHARP.GND
- net INT0: now also IC3.INT1
- net INT1: now also IC3.INT2; no longer IC3.INT1
- net MISO: now also ISP1.1; no longer ICSP.1
- net MOSI: no longer ICSP.4
- net PROXIN: now also JP3.1; no longer JP5.1, SHARP.VOUT
- net RESET: now also ISP1.5, SJ3.2; no longer ICSP.5, RESET.1, RESET.2
- net RXD: now also JP5.TXO; no longer JP4.TXO
- net SCK: now also ISP1.3; no longer ICSP.3
- net TXD: now also JP5.RXI; no longer JP4.RXI
- net V+: now also C7.1; no longer JP1.1, JP7.1
- net VIBE: no longer JP7.2
- net VIBE_CONTROL: now also IC4.PD4(XCK/T0); no longer IC4.PB0(ICP)
Other:
- moved on the sheet: JP6

Commit message: All routed except for LEDs (which will be hard)
Parts:
- removed LED2: (no value), led:LEDCHIPLED_0805
- removed R6: 470, rcl:R-US_R0603
- added R8, R9: 4.7k, rcl:R-US_R0603
Connections:
- removed net N$4: LED2.A, R6.1
- net +3V3: now also ISP1.2, R8.2, R9.2
- net GND: now also ISP1.6; no longer LED2.C
- net GREEN: now also IC4.PB1(OC1A); no longer IC4.PD5(T1)
- net MOSI: now also ISP1.4
- net RED: now also IC4.PD5(T1); no longer IC4.PB1(OC1A)
- net SCL: now also R9.1
- net SDA: now also R8.1
- net STATUS: no longer R6.2
Changed lines of the file:
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@@
 <part name="GND2" library="supply1" deviceset="GND" device=""/>
 <part name="IC4" library="SparkFun" deviceset="ATMEGA168" device=""/>
-<part name="LED2" library="led" deviceset="LED" device="CHIPLED_0805"/>
 <part name="C13" library="rcl" deviceset="C-US" device="C0603" value="10uF"/>
 <part name="C14" library="rcl" deviceset="C-US" device="C0603" value=".1uF"/>
@@
 <part name="R7" library="rcl" deviceset="R-US_" device="R0603" value="10k"/>
 <part name="+3V4" library="supply1" deviceset="+3V3" device=""/>
-<part name="R6" library="rcl" deviceset="R-US_" device="R0603" value="470"/>
 <part name="GND5" library="supply1" deviceset="GND" device=""/>
 <part name="GND6" library="supply1" deviceset="GND" device=""/>
@@
 <part name="T2" library="transistor" deviceset="*-NPN-" device="SOT23-EBC"/>
 <part name="GND11" library="supply1" deviceset="GND" device=""/>
-<part name="GND3" library="supply1" deviceset="GND" device=""/>
 <part name="LED1" library="led" deviceset="LED" device="CHIPLED_0805"/>
 <part name="R5" library="rcl" deviceset="R-US_" device="R0603" value="470"/>
@@
 <part name="GND13" library="supply1" deviceset="GND" device=""/>
 <part name="SJ3" library="SparkFun" deviceset="SOLDERJUMPER" device="NO"/>
+<part name="R8" library="rcl" deviceset="R-US_" device="R0603" value="4.7k"/>
+<part name="R9" library="rcl" deviceset="R-US_" device="R0603" value="4.7k"/>
+<part name="+3V14" library="supply1" deviceset="+3V3" device=""/>
+<part name="+3V15" library="supply1" deviceset="+3V3" device=""/>
 </parts>
 <sheets>
@@
 -Do we want a PMC?
 -Check pin layout power consump for LED Driver
--Check MSOP spacing with a print out</text>
+-Check MSOP spacing with a print out
+-Check i2C pullups</text>
 </plain>
 <instances>
@@
 <instance part="GND2" gate="1" x="497.84" y="322.58"/>
 <instance part="IC4" gate="G$1" x="259.08" y="78.74"/>
-<instance part="LED2" gate="G$1" x="269.24" y="210.82"/>
 <instance part="C13" gate="G$1" x="205.74" y="76.2"/>
 <instance part="C14" gate="G$1" x="215.9" y="76.2"/>
@@
 <instance part="R7" gate="G$1" x="233.68" y="114.3" rot="R90"/>
 <instance part="+3V4" gate="G$1" x="205.74" y="104.14"/>
-<instance part="R6" gate="G$1" x="269.24" y="218.44" rot="R90"/>
 <instance part="GND5" gate="1" x="215.9" y="66.04"/>
 <instance part="GND6" gate="1" x="205.74" y="66.04"/>
@@
 <instance part="T2" gate="G$1" x="86.36" y="104.14"/>
 <instance part="GND11" gate="1" x="218.44" y="337.82"/>
-<instance part="GND3" gate="1" x="269.24" y="200.66"/>
 <instance part="LED1" gate="G$1" x="259.08" y="210.82"/>
 <instance part="R5" gate="G$1" x="259.08" y="218.44" rot="R90"/>
@@
 <instance part="GND13" gate="1" x="538.48" y="81.28"/>
 <instance part="SJ3" gate="1" x="213.36" y="231.14" rot="R180"/>
+<instance part="R8" gate="G$1" x="408.94" y="233.68" rot="R90"/>
+<instance part="R9" gate="G$1" x="401.32" y="233.68" rot="R90"/>
+<instance part="+3V14" gate="G$1" x="408.94" y="243.84"/>
+<instance part="+3V15" gate="G$1" x="401.32" y="243.84"/>
 </instances>
 <busses>
@@
 <pinref part="GND5" gate="1" pin="GND"/>
 <wire x1="215.9" y1="71.12" x2="215.9" y2="68.58" width="0.1524" layer="91"/>
-</segment>
-<segment>
-<wire x1="215.9" y1="195.58" x2="223.52" y2="195.58" width="0.1524" layer="91"/>
-<pinref part="GND7" gate="1" pin="GND"/>
-<wire x1="223.52" y1="195.58" x2="223.52" y2="193.04" width="0.1524" layer="91"/>
 </segment>
 <segment>
@@
 <junction x="200.66" y="342.9"/>
 <wire x1="218.44" y1="342.9" x2="236.22" y2="342.9" width="0.1524" layer="91"/>
-</segment>
-<segment>
-<pinref part="LED2" gate="G$1" pin="C"/>
-<wire x1="269.24" y1="205.74" x2="269.24" y2="203.2" width="0.1524" layer="91"/>
-<pinref part="GND3" gate="1" pin="GND"/>
 </segment>
 <segment>
@@
 <wire x1="538.48" y1="83.82" x2="538.48" y2="88.9" width="0.1524" layer="91"/>
 </segment>
+<segment>
+<pinref part="ISP1" gate="A" pin="6"/>
+<pinref part="GND7" gate="1" pin="GND"/>
+<wire x1="215.9" y1="195.58" x2="223.52" y2="195.58" width="0.1524" layer="91"/>
+<wire x1="223.52" y1="195.58" x2="223.52" y2="193.04" width="0.1524" layer="91"/>
+</segment>
 </net>
 <net name="+3V3" class="0">
@@
 </segment>
 <segment>
-<wire x1="215.9" y1="200.66" x2="223.52" y2="200.66" width="0.1524" layer="91"/>
-<pinref part="+3V7" gate="G$1" pin="+3V3"/>
-<wire x1="223.52" y1="200.66" x2="223.52" y2="205.74" width="0.1524" layer="91"/>
-</segment>
-<segment>
 <wire x1="317.5" y1="218.44" x2="304.8" y2="218.44" width="0.1524" layer="91"/>
 <pinref part="+3V8" gate="G$1" pin="+3V3"/>
@@
 <wire x1="269.24" y1="363.22" x2="269.24" y2="368.3" width="0.1524" layer="91"/>
 <pinref part="C4" gate="G$1" pin="1"/>
+</segment>
+<segment>
+<pinref part="+3V15" gate="G$1" pin="+3V3"/>
+<pinref part="R9" gate="G$1" pin="2"/>
+<wire x1="401.32" y1="241.3" x2="401.32" y2="238.76" width="0.1524" layer="91"/>
+</segment>
+<segment>
+<pinref part="+3V14" gate="G$1" pin="+3V3"/>
+<pinref part="R8" gate="G$1" pin="2"/>
+<wire x1="408.94" y1="241.3" x2="408.94" y2="238.76" width="0.1524" layer="91"/>
+</segment>
+<segment>
+<pinref part="ISP1" gate="A" pin="2"/>
+<pinref part="+3V7" gate="G$1" pin="+3V3"/>
+<wire x1="215.9" y1="200.66" x2="223.52" y2="200.66" width="0.1524" layer="91"/>
+<wire x1="223.52" y1="200.66" x2="223.52" y2="205.74" width="0.1524" layer="91"/>
 </segment>
 </net>
@@
 <net name="STATUS" class="0">
 <segment>
-<pinref part="R6" gate="G$1" pin="2"/>
-<wire x1="269.24" y1="226.06" x2="269.24" y2="223.52" width="0.1524" layer="91"/>
-<label x="269.24" y="226.06" size="1.27" layer="95" font="vector" ratio="15" rot="R90" xref="yes"/>
-</segment>
-<segment>
 <pinref part="IC4" gate="G$1" pin="PD7(AIN1)"/>
 <wire x1="284.48" y1="63.5" x2="289.56" y2="63.5" width="0.1524" layer="91"/>
@@
 </segment>
 </net>
-<net name="N$4" class="0">
-<segment>
-<pinref part="LED2" gate="G$1" pin="A"/>
-<pinref part="R6" gate="G$1" pin="1"/>
-</segment>
-</net>
 <net name="MOSI" class="0">
-<segment>
-<wire x1="215.9" y1="198.12" x2="223.52" y2="198.12" width="0.1524" layer="91"/>
-<label x="223.52" y="198.12" size="1.27" layer="95" font="vector" ratio="15" xref="yes"/>
-</segment>
 <segment>
 <pinref part="IC4" gate="G$1" pin="PB3(MOSI/OC2)"/>
@@
 <label x="289.56" y="50.8" size="1.27" layer="95" font="vector" ratio="15" xref="yes"/>
 </segment>
+<segment>
+<pinref part="ISP1" gate="A" pin="4"/>
+<wire x1="215.9" y1="198.12" x2="226.06" y2="198.12" width="0.1524" layer="91"/>
+<label x="226.06" y="198.12" size="1.27" layer="95" font="vector" ratio="14" xref="yes"/>
+</segment>
 </net>
 <net name="MISO" class="0">
@@
 <net name="RED" class="0">
 <segment>
-<pinref part="IC4" gate="G$1" pin="PB1(OC1A)"/>
-<wire x1="284.48" y1="55.88" x2="289.56" y2="55.88" width="0.1524" layer="91"/>
-<label x="289.56" y="55.88" size="1.27" layer="95" font="vector" ratio="15" xref="yes"/>
-</segment>
-<segment>
 <pinref part="IC6" gate="G$1" pin="IN3"/>
 <wire x1="464.82" y1="88.9" x2="474.98" y2="88.9" width="0.1524" layer="91"/>
 <label x="464.82" y="88.9" size="1.27" layer="95" font="vector" ratio="15" rot="R180" xref="yes"/>
+</segment>
+<segment>
+<pinref part="IC4" gate="G$1" pin="PD5(T1)"/>
+<wire x1="284.48" y1="68.58" x2="289.56" y2="68.58" width="0.1524" layer="91"/>
+<label x="289.56" y="68.58" size="1.27" layer="95" font="vector" ratio="15" xref="yes"/>
 </segment>
 </net>
@@
 <net name="SCL" class="0">
 <segment>
-<wire x1="441.96" y1="220.98" x2="419.1" y2="220.98" width="0.1524" layer="91"/>
-<label x="419.1" y="220.98" size="1.27" layer="95" font="vector" ratio="15" rot="R180" xref="yes"/>
+<wire x1="441.96" y1="220.98" x2="401.32" y2="220.98" width="0.1524" layer="91"/>
+<label x="393.7" y="220.98" size="1.27" layer="95" font="vector" ratio="15" rot="R180" xref="yes"/>
 <pinref part="IC3" gate="G$1" pin="SCL"/>
+<pinref part="R9" gate="G$1" pin="1"/>
+<wire x1="401.32" y1="220.98" x2="393.7" y2="220.98" width="0.1524" layer="91"/>
+<wire x1="401.32" y1="228.6" x2="401.32" y2="220.98" width="0.1524" layer="91"/>
+<junction x="401.32" y="220.98"/>
 </segment>
 <segment>
@@
 <net name="SDA" class="0">
 <segment>
-<wire x1="441.96" y1="223.52" x2="419.1" y2="223.52" width="0.1524" layer="91"/>
-<label x="419.1" y="223.52" size="1.27" layer="95" font="vector" ratio="15" rot="R180" xref="yes"/>
+<wire x1="441.96" y1="223.52" x2="408.94" y2="223.52" width="0.1524" layer="91"/>
+<label x="393.7" y="223.52" size="1.27" layer="95" font="vector" ratio="15" rot="R180" xref="yes"/>
 <pinref part="IC3" gate="G$1" pin="SDA"/>
+<pinref part="R8" gate="G$1" pin="1"/>
+<wire x1="408.94" y1="223.52" x2="393.7" y2="223.52" width="0.1524" layer="91"/>
+<wire x1="408.94" y1="228.6" x2="408.94" y2="223.52" width="0.1524" layer="91"/>
+<junction x="408.94" y="223.52"/>
 </segment>
 <segment>
@@
 <net name="GREEN" class="0">
 <segment>
-<pinref part="IC4" gate="G$1" pin="PD5(T1)"/>
-<wire x1="284.48" y1="68.58" x2="289.56" y2="68.58" width="0.1524" layer="91"/>
-<label x="289.56" y="68.58" size="1.27" layer="95" font="vector" ratio="15" xref="yes"/>
-</segment>
-<segment>
 <pinref part="IC6" gate="G$1" pin="IN2"/>
 <wire x1="474.98" y1="93.98" x2="464.82" y2="93.98" width="0.1524" layer="91"/>
 <label x="464.82" y="93.98" size="1.27" layer="95" font="vector" ratio="15" rot="R180" xref="yes"/>
 </segment>
-</net>
+<segment>
+<pinref part="IC4" gate="G$1" pin="PB1(OC1A)"/>
+<wire x1="284.48" y1="55.88" x2="289.56" y2="55.88" width="0.1524" layer="91"/>
+<label x="289.56" y="55.88" size="1.27" layer="95" font="vector" ratio="15" xref="yes"/>
+</segment>
+</net>
